Commit message: 10/12

File: xArm/xarm_description/urdf/HappyDaisy.urdf.xacro (robot description, xacro)
@@ -34,17 +34,17 @@
       <visual>
         <geometry>
-          <mesh filename="package://xarm_description/meshes/HappyDaisy/HappyDaisy.dae"/>
+            <mesh filename="package://xarm_description/meshes/HappyDaisy/mrp_v43.stl" scale="0.001 0.001 0.001"/>
           <!--mesh filename="package://xarm_description/meshes/HappyDaisy/WRS_hard.dae"/-->
           <!--mesh filename="package://xarm_description/meshes/HappyDaisy/HappyDaisy.stl" scale="0.001 0.001 0.001"/-->
         </geometry>
-        <origin xyz="0 0 0" rpy="0 0 0"/>
-      </visual>
-      <collision>
-        <geometry>
-          <mesh filename="package://xarm_description/meshes/HappyDaisy/HappyDaisy.dae"/>
+        <origin xyz="0 0 0" rpy="1.57 0 0"/>
+      </visual>
+      <collision>
+        <geometry>
+            <mesh filename="package://xarm_description/meshes/HappyDaisy/mrp_v43.stl" scale="0.001 0.001 0.001"/>
           <!--mesh filename="package://xarm_description/meshes/HappyDaisy/WRS_hard.dae"/-->
           <!--mesh filename="package://xarm_description/meshes/HappyDaisy/HappyDaisy.stl"/-->
         </geometry>
-        <origin xyz="0 0 0" rpy="0 0 0"/>
+        <origin xyz="0 0 0" rpy="1.57 0 0"/>
       </collision>
     </link>
