Commit message: competition

File: xArm/xarm_description/urdf/xarm6_robot_macro.xacro (robot description, xacro)
@@ -13,5 +13,5 @@
     geometry_mesh_tcp_rpy:='0 0 0' ">
     <!-- include xarm6 relative macros: -->
-    <!-- xacro:include filename="$(find xarm_description)/urdf/xarm6.urdf.xacro" /-->
+    <!--xacro:include filename="$(find xarm_description)/urdf/xarm6.urdf.xacro" /-->
     <xacro:include filename="$(find xarm_description)/urdf/HappyDaisy.urdf.xacro" />
     <xacro:include filename="$(find xarm_description)/urdf/xarm6.transmission.xacro" />

File: xArm/xarm_description/urdf/xarm_vacuum_gripper.urdf.xacro (robot description, xacro)
@@ -31,24 +31,27 @@
     </inertial>
     <visual>
+      <!--origin
+        xyz="0.006 0 -0.012"
+        rpy="-1.57 3.14 0" /-->
       <origin
-        xyz="0.006 0 0.038"
-        rpy="-1.57 3.14 0" />
+        xyz="0.006 0 -0.012"
+        rpy="-1.57 3.14 -0.2" />
       <geometry>
         <!--mesh
           filename="package://xarm_description/meshes/vacuum_gripper/visual/vacuum_gripper.STL" /-->
-        <mesh filename="package://xarm_description/meshes/vacuum_gripper/visual/end_effector.stl" scale="0.001 0.001 0.001"/>
+        <mesh filename="package://xarm_description/meshes/vacuum_gripper/visual/short_endeffector.stl" scale="0.001 0.001 0.001"/>
       </geometry>
       <material name="White">
-        <color rgba="1.0 1.0 1.0 1.0"/>
+        <color rgba="1.0 1.0 0 1.0"/>
       </material>
     </visual>
     <collision>
       <origin
-        xyz="0 0 0"
-        rpy="0 0 0" />
+          xyz="0.006 0 -0.012"
+          rpy="-1.57 3.14 -0.2" />
       <geometry>
         <!--mesh
           filename="package://xarm_description/meshes/vacuum_gripper/collision/vacuum_gripper.STL" /-->
-        <mesh filename="package://xarm_description/meshes/vacuum_gripper/collision/end_effector.stl" scale="0.001 0.001 0.001"/>
+        <mesh filename="package://xarm_description/meshes/vacuum_gripper/collision/short_endeffector.stl" scale="0.001 0.001 0.001"/>
       </geometry>
     </collision>
@@ -58,6 +61,12 @@
     name="${prefix}joint_tcp"
     type="fixed">
-    <origin
+    <!--origin
       xyz="0 0 0.126"
+      rpy="0 0 0" /-->
+    <!--origin
+      xyz="0 0.02 0.2"
+      rpy="0 0 0" /-->
+       <origin
+      xyz="-0.0017 0.0237 0.2"
       rpy="0 0 0" />
     <parent
@@ -66,4 +75,28 @@
       link="${prefix}link_tcp" />
   </joint>
+  <!--link name="${prefix}link_tcp2" />
+  <joint
+    name="${prefix}joint_tcp2"
+    type="fixed">
+    <origin
+      xyz="0 0.03 0.2"
+      rpy="0 0 0" />
+    <parent
+      link="${prefix}xarm_vacuum_gripper_link" />
+    <child
+      link="${prefix}link_tcp2" />
+  </joint>
+  <link name="${prefix}link_tcp3" />
+  <joint
+    name="${prefix}joint_tcp3"
+    type="fixed">
+    <origin
+      xyz="0 0.03 0.2"
+      rpy="0 0 0" />
+    <parent
+      link="${prefix}xarm_vacuum_gripper_link" />
+    <child
+      link="${prefix}link_tcp3" />
+  </joint-->
   </xacro:macro>
 </robot>
